File: src/microscope-lamp-pcb/microscope-lamp-pcb.kicad_pcb (KiCad board)
At the start: 2 copper layers, 34 x 45 mm, 31 parts, among them J1 USB_C_Receptacle_PowerOnly_6P, U1 AP5724WG

Commit message: removing OSH logo
Parts:
- removed REF**: OSHW-Logo2_7.3x6mm_SilkScreen, Symbol:OSHW-Logo2_7.3x6mm_SilkScreen
Other:
- board text added: "open source hardware"
